Commit message: fix name error

File: rosaya/urdf/rosaya.urdf (robot description, URDF)
Before this commit: robot rosaya, 15 links, 14 joints
Links:
- removed link L-Link
- removed link L-Link1
- removed link L-Link2
- removed link L-Link3
- removed link L-Link4
- removed link L-Link5
- removed link R-Link
- removed link R-Link1
- removed link R-Link2
- removed link R-Link3
- removed link R-Link4
- removed link R-Link5
- added link L_Link, mass 0.0062048; collision mesh filename=package://rosaya/meshes/L_Link.STL; visual mesh filename=package://rosaya/meshes/L_Link.STL
- added link L_Link1, mass 0.186396401372013; collision mesh filename=package://rosaya/meshes/L_Link1.STL; visual mesh filename=package://rosaya/meshes/L_Link1.STL
- added link L_Link2, mass 0.099079; collision mesh filename=package://rosaya/meshes/L_Link2.STL; visual mesh filename=package://rosaya/meshes/L_Link2.STL
- added link L_Link3, mass 0.0193582268613659; collision mesh filename=package://rosaya/meshes/L_Link3.STL; visual mesh filename=package://rosaya/meshes/L_Link3.STL
- added link L_Link4, mass 0.18164; collision mesh filename=package://rosaya/meshes/L_Link4.STL; visual mesh filename=package://rosaya/meshes/L_Link4.STL
- added link L_Link5, mass 0.072891; collision mesh filename=package://rosaya/meshes/L_Link5.STL; visual mesh filename=package://rosaya/meshes/L_Link5.STL
- added link R_Link, mass 0.0062048; collision mesh filename=package://rosaya/meshes/R_Link.STL; visual mesh filename=package://rosaya/meshes/R_Link.STL
- added link R_Link1, mass 0.1864; collision mesh filename=package://rosaya/meshes/R_Link1.STL; visual mesh filename=package://rosaya/meshes/R_Link1.STL
- added link R_Link2, mass 0.099079; collision mesh filename=package://rosaya/meshes/R_Link2.STL; visual mesh filename=package://rosaya/meshes/R_Link2.STL
- added link R_Link3, mass 0.019358; collision mesh filename=package://rosaya/meshes/R_Link3.STL; visual mesh filename=package://rosaya/meshes/R_Link3.STL
- added link R_Link4, mass 0.18164; collision mesh filename=package://rosaya/meshes/R_Link4.STL; visual mesh filename=package://rosaya/meshes/R_Link4.STL
- added link R_Link5, mass 0.072891; collision mesh filename=package://rosaya/meshes/R_Link5.STL; visual mesh filename=package://rosaya/meshes/R_Link5.STL
- link Link1: mass 0.264483114754865 -> 0.26448
- link Link2: mass 0.266759815938641 -> 0.26676
- link Link3: mass 0.141461102552141 -> 0.14146
Joints:
- joint Joint10: child R-Link3 -> R_Link3; parent R-Link2 -> R_Link2
- joint Joint11: child L-Link4 -> L_Link4; parent L-Link3 -> L_Link3
- joint Joint12: child R-Link4 -> R_Link4; parent R-Link3 -> R_Link3
- joint Joint13: child L-Link5 -> L_Link5; parent L-Link4 -> L_Link4
- joint Joint14: child R-Link5 -> R_Link5; parent R-Link4 -> R_Link4
- joint Joint3: child L-Link -> L_Link
- joint Joint4: child R-Link -> R_Link
- joint Joint5: child L-Link1 -> L_Link1; origin xyz=-0.0294500000000014 0 -0.0339141545469447 rpy=0.000537539761406673 0 0 -> xyz=-0.0317500000000014 0 -0.0339141545469447 rpy=0.000537539761406673 0 0; parent L-Link -> L_Link
- joint Joint6: child R-Link1 -> R_Link1; parent R-Link -> R_Link
- joint Joint7: child L-Link2 -> L_Link2; origin xyz=0.0294200000000001 -0.0244999999999996 0 rpy=0 0 0 -> xyz=0.0317200000000001 -0.0244999999999996 0 rpy=0 0 0; parent L-Link1 -> L_Link1
- joint Joint8: child R-Link2 -> R_Link2; parent R-Link1 -> R_Link1
- joint Joint9: child L-Link3 -> L_Link3; parent L-Link2 -> L_Link2
