Commit message: Merged new code

File: rosaya_moveit/config/gazebo_rosaya_models.urdf (robot description, URDF)
Before this commit: robot rosaya, 15 links, 14 joints
Links:
- link L_Link: mass 0.0062048 -> 0.00620476919773645
- link L_Link1: mass 0.186396401372013 -> 0.18639489707273
- link L_Link2: mass 0.099079 -> 0.0990788181499382
- link L_Link4: mass 0.18164 -> 0.182895656171114
- link L_Link5: mass 0.072891 -> 0.0728910331350744
- link Link1: mass 0.26448 -> 0.264483114754865
- link Link2: mass 0.26676 -> 0.266759815938641
- link Link3: mass 0.14146 -> 0.141461102552141
- link R_Link: mass 0.0062048 -> 0.00620476919773645
- link R_Link1: mass 0.1864 -> 0.18639489707273
- link R_Link2: mass 0.099079 -> 0.0990788181535519
- link R_Link3: mass 0.019358 -> 0.0193582268613659
- link R_Link4: mass 0.18164 -> 0.182895656171117
- link R_Link5: mass 0.072891 -> 0.0728910331350756
Joints:
- joint Joint1: axis 1 0 0 -> -1 0 0; origin xyz=0.0150416145062784 -0.000145225937100715 0.375282029235617 rpy=-0.00310746977134566 0 0 -> xyz=0.0150416145062784 -0.000145225937100715 0.375282029235617 rpy=0.00310746977134566 0 -3.14159265358979
- joint Joint10: axis 0 1 0 -> 0 -1 0; origin xyz=0 0.0014000000000008 -0.11278054553733 rpy=0 0 0 -> xyz=0 -0.0014000000000008 -0.11278054553733 rpy=0 0 0
- joint Joint11: axis 0 1 0 -> 0 -1 0; origin xyz=0 0 -0.0949999999999996 rpy=0 0.000302748335169453 0 -> xyz=0 0 -0.0949999999999996 rpy=0 -0.000302748335169453 3.14159265358979
- joint Joint12: origin xyz=0 0 -0.0949999999999999 rpy=0 0 0 -> xyz=0 0 -0.0949999999999999 rpy=0 0 3.14159265358979
- joint Joint13: axis 1 0 0 -> -1 0 0; origin xyz=-0.0236 0.026 0 rpy=0 0 0 -> xyz=0.0235999999999932 -0.0259999999999994 0 rpy=0 0 0
- joint Joint14: axis 1 0 0 -> -1 0 0; origin xyz=-0.0235999999999946 -0.0260000000000017 0 rpy=0 0 0 -> xyz=-0.0235999999999946 -0.0260000000000017 0 rpy=0 0 3.14159265358979
- joint Joint2: origin xyz=-0.0150417125919951 0.000171249925764887 -0.0551096819554042 rpy=0.00310746977134566 0 0 -> xyz=0.0150417125919951 -0.00017124992576488 -0.0551096819554042 rpy=0.00310746977134566 0 3.14159265358979
- joint Joint8: axis 0 1 0 -> 0 -1 0; origin xyz=0.031720000000165 0.0245000000000003 -4.90873395437297E-05 rpy=0 0 0 -> xyz=0.031720000000165 0.0245000000000003 -4.90873395437297E-05 rpy=0 0 -3.14159265358979

Commit message: Update motion

File: rosaya_moveit/config/gazebo_rosaya_models.urdf (robot description, URDF)
Before this commit: robot rosaya_models, 15 links, 14 joints
Joints:
- joint Joint1: limit (none) -> lower=-1 upper=1 effort=0 velocity=0; type continuous -> revolute
- joint Joint10: limit (none) -> lower=-0.5 upper=2.5 effort=0 velocity=0; type continuous -> revolute
- joint Joint11: limit (none) -> lower=-2. upper=1 effort=0 velocity=0; type continuous -> revolute
- joint Joint12: axis 0 1 0 -> 0 -1 0; limit (none) -> lower=-1 upper=2 effort=0 velocity=0; type continuous -> revolute
- joint Joint13: limit (none) -> lower=-2 upper=2 effort=0 velocity=0; type continuous -> revolute
- joint Joint14: limit (none) -> lower=-2 upper=2 effort=0 velocity=0; type continuous -> revolute
- joint Joint2: axis 0 0 1 -> 0 0 -1; limit (none) -> lower=-2 upper=2 effort=0 velocity=0; type continuous -> revolute
- joint Joint3: axis 0 0 1 -> 0 0 -1; limit (none) -> lower=-1 upper=1 effort=0 velocity=0; type continuous -> revolute
- joint Joint4: axis 0 0 1 -> 0 0 -1; limit (none) -> lower=-1 upper=1 effort=0 velocity=0; type continuous -> revolute
- joint Joint5: axis 1 0 0 -> -1 0 0; limit (none) -> lower=-0.7 upper=0.7 effort=0 velocity=0; type continuous -> revolute
- joint Joint6: axis 1 0 0 -> -1 0 0; limit (none) -> lower=-0.7 upper=0.7 effort=0 velocity=0; type continuous -> revolute
- joint Joint7: axis 0 1 0 -> 0 -1 0; limit (none) -> lower=-0.8 upper=2 effort=0 velocity=0; type continuous -> revolute
- joint Joint8: limit (none) -> lower=-2 upper=0.8 effort=0 velocity=0; type continuous -> revolute
- joint Joint9: axis 0 1 0 -> 0 -1 0; limit (none) -> lower=-2.5 upper=0.5 effort=0 velocity=0; type continuous -> revolute
