Commit message: Update configuration

File: rosaya_models/urdf/rosaya_models.urdf (robot description, URDF)
Before this commit: robot rosaya_models, 15 links, 14 joints
Joints:
- joint Joint13: limit lower=-2 upper=2 effort=0 velocity=0 -> lower=-0.6 upper=0.6 effort=0 velocity=0
- joint Joint14: limit lower=-2 upper=2 effort=0 velocity=0 -> lower=-0.6 upper=0.6 effort=0 velocity=0

File: rosaya_moveit/config/gazebo_rosaya_models.urdf (robot description, URDF)
Before this commit: robot rosaya_models, 15 links, 14 joints
Joints:
- joint Joint13: limit lower=-2 upper=2 effort=0 velocity=0 -> lower=-0.6 upper=0.6 effort=0 velocity=0
- joint Joint14: limit lower=-2 upper=2 effort=0 velocity=0 -> lower=-0.6 upper=0.6 effort=0 velocity=0
